Commit message: Added ros control and fixed gazebo plugin bugs

File: my_robot_description/urdf/mobile_base.xacro (robot description, xacro)
@@ -54,4 +54,15 @@
         </inertial>
       </link>
+      <!-- <link name="steering_wheel_link">
+        <visual>
+            <geometry>
+                <cylinder radius="${wheel_radius}" length="${wheel_length}" />
+            </geometry>
+            <origin xyz="0 0 0" rpy="${pi / 2.0} 0 0" />
+            <material name="grey" />
+        </visual>
+        <xacro:cylinder_inertia m="${wheel_mass}" r="${2*wheel_radius}" l="${2*wheel_length}"
+                                xyz="0 0 0" rpy="0 0 0" />
+    </link>-->
     <!--JOINT-->
     <joint name="base_joint" type="fixed">
@@ -103,16 +114,12 @@
         <axis xyz="0 1 0" />
     </joint>
-    <!--STEERING WHEEL JOINT-->
-    <link name="steering_wheel">
-        <mass value="0.1" />
-        <inertia ixx="1.0" ixy="0.0" ixz="0.0" iyy="1.0" iyz="0.0" izz="1.0" />
-    </link>
+    <!--STEERING WHEEL JOINT
     <joint name="steering_joint" type="revolute">
         <parent link="base_link" />
-        <child link="steering_wheel" />
+        <child link="steering_wheel_link" />
         <origin xyz="${base_length / 4.0} 0 0" rpy="0 0 0"/>
         <axis xyz="0.0 0.0 1.0" />
         <dynamics damping="0.01" friction="0.01" />
         <limit effort="1000.0" lower="-0.95" upper="0.95" velocity="100" />
-    </joint>
+    </joint>-->
 </robot>

File: my_robot_description/urdf/mobile_base_gazebo.xacro (robot description, xacro)
@@ -13,37 +13,43 @@
     <xacro:wheel_gazebo prefix="back_l" />
     <xacro:wheel_gazebo prefix="back_r" />
-    <gazebo>
-        <plugin name='ackermann_drive' filename='libgazebo_ros_ackermann_drive.so'>
-            <update_rate>100.0</update_rate>
-            <!-- wheels -->
-            <front_left_joint>l_steer_front_l_wheel_joint</front_left_joint>
-            <front_right_joint>r_steer_front_r_wheel_joint</front_right_joint>
-            <rear_left_joint>base_back_l_wheel_joint</rear_left_joint>
-            <rear_right_joint>base_back_r_wheel_joint</rear_right_joint>
-            <left_steering_joint>base_l_steer_joint</left_steering_joint>
-            <right_steering_joint>base_r_steer_joint</right_steering_joint>
-            <steering_wheel_joint>steering_joint</steering_wheel_joint>
-            <!-- Max absolute steer angle for tyre in radians-->
-            <!-- Any cmd_vel angular z greater than this would be capped -->
-            <max_steer>0.6458</max_steer>
-            <!-- Max absolute steering angle of steering wheel -->
-            <max_steering_angle>7.85</max_steering_angle>
-            <!-- Max absolute linear speed in m/s -->
-            <max_speed>20</max_speed>
-            <!-- PID tuning -->
-            <left_steering_pid_gain>1500 0 1</left_steering_pid_gain>
-            <left_steering_i_range>0 0</left_steering_i_range>
-            <right_steering_pid_gain>1500 0 1</right_steering_pid_gain>
-            <right_steering_i_range>0 0</right_steering_i_range>
-            <linear_velocity_pid_gain>1000 0 1</linear_velocity_pid_gain>
-            <linear_velocity_i_range>0 0</linear_velocity_i_range>
-            <!-- output -->
-            <publish_odom>true</publish_odom>
-            <publish_odom_tf>true</publish_odom_tf>
-            <publish_wheel_tf>true</publish_wheel_tf>
-            <publish_distance>true</publish_distance>
-            <odometry_frame>odom</odometry_frame>
-            <robot_base_frame>base_footprint</robot_base_frame>
-        </plugin>
-    </gazebo>
+    <!-- <xacro:wheel_gazebo prefix="steering" />-->
+     <!-- Ackermann driver -->
+  <ros2_control name="GazeboSystem" type="system">
+    <hardware>
+      <plugin>gazebo_ros2_control/GazeboSystem</plugin>
+    </hardware>
+    <joint name="base_back_l_wheel_joint">
+      <command_interface name="velocity"/>
+      <state_interface name="position"/>
+      <state_interface name="velocity"/>
+    </joint>
+    <joint name="base_back_r_wheel_joint">
+      <command_interface name="velocity"/>
+      <state_interface name="position"/>
+      <state_interface name="velocity"/>
+    </joint>
+    <joint name="base_l_steer_joint">
+      <command_interface name="position"/>
+      <state_interface name="position"/>
+      <state_interface name="velocity"/>
+    </joint>
+    <joint name="base_r_steer_joint">
+      <command_interface name="position"/>
+      <state_interface name="position"/>
+      <state_interface name="velocity"/>
+    </joint>
+    <!-- <joint name="l_steer_front_l_wheel_joint">
+      <state_interface name="position"/>
+      <state_interface name="velocity"/>
+    </joint>
+    <joint name="r_steer_front_r_wheel_joint">
+      <state_interface name="position"/>
+      <state_interface name="velocity"/>
+    </joint>-->
+  </ros2_control>
+  <gazebo>
+    <plugin name="gazebo_ros2_control" filename="libgazebo_ros2_control.so">
+        <parameters>$(find my_robot_bringup)/config/ackermann_config.yaml</parameters>
+    </plugin>
+  </gazebo>
 </robot>

Commit message: Added ros2 control spawner inside the launch file

File: my_robot_description/urdf/mobile_base.xacro (robot description, xacro)
@@ -54,15 +54,4 @@
         </inertial>
       </link>
-      <!-- <link name="steering_wheel_link">
-        <visual>
-            <geometry>
-                <cylinder radius="${wheel_radius}" length="${wheel_length}" />
-            </geometry>
-            <origin xyz="0 0 0" rpy="${pi / 2.0} 0 0" />
-            <material name="grey" />
-        </visual>
-        <xacro:cylinder_inertia m="${wheel_mass}" r="${2*wheel_radius}" l="${2*wheel_length}"
-                                xyz="0 0 0" rpy="0 0 0" />
-    </link>-->
     <!--JOINT-->
     <joint name="base_joint" type="fixed">
@@ -114,12 +103,3 @@
         <axis xyz="0 1 0" />
     </joint>
-    <!--STEERING WHEEL JOINT
-    <joint name="steering_joint" type="revolute">
-        <parent link="base_link" />
-        <child link="steering_wheel_link" />
-        <origin xyz="${base_length / 4.0} 0 0" rpy="0 0 0"/>
-        <axis xyz="0.0 0.0 1.0" />
-        <dynamics damping="0.01" friction="0.01" />
-        <limit effort="1000.0" lower="-0.95" upper="0.95" velocity="100" />
-    </joint>-->
 </robot>
