Commit message: Added front wheels in ros2_control plugin

File: my_robot_description/urdf/mobile_base_gazebo.xacro (robot description, xacro)
@@ -39,12 +39,15 @@
       <state_interface name="velocity"/>
     </joint>
-    <!-- <joint name="l_steer_front_l_wheel_joint">
+    <!--FRONT WHEEL-->
+    <joint name="l_steer_front_l_wheel_joint">
       <state_interface name="position"/>
       <state_interface name="velocity"/>
+      <state_interface name="effort"/>
     </joint>
     <joint name="r_steer_front_r_wheel_joint">
       <state_interface name="position"/>
       <state_interface name="velocity"/>
-    </joint>-->
+      <state_interface name="effort"/>
+    </joint>
   </ros2_control>
   <gazebo>
